Commit message: Add RS02 firmware compatibility and recovery

File: robstride_examples/description/robstride_example.urdf.xacro (robot description, xacro)
@@ -21,5 +21,5 @@
       <param name="fail_on_feedback_timeout">true</param>
       <param name="transmit_failure_timeout_ms">1000</param>
-      <param name="run_mode_recovery_timeout_ms">500</param>
+      <param name="run_mode_recovery_timeout_ms">10000</param>
       <param name="run_mode_recovery_retry_interval_ms">100</param>
       <param name="clear_faults_on_activate">true</param>
@@ -33,5 +33,5 @@
     </hardware>
     <joint name="robstride_joint">
-      <xacro:robstride_edulite05_params can_id="1" direction="1" kp="30.0" kd="1.0"/>
+      <xacro:robstride_rs02_params can_id="4" direction="1" kp="30.0" kd="1.0"/>
       <xacro:robstride_joint_interfaces/>
     </joint>

File: robstride_ros2_control/description/robstride_motor_profiles.xacro (robot description, xacro)
@@ -35,5 +35,5 @@
     <xacro:robstride_command_limits position_min="${command_position_min}" position_max="${command_position_max}" velocity_min="${command_velocity_min}" velocity_max="${command_velocity_max}" effort_min="${command_effort_min}" effort_max="${command_effort_max}"/>
   </xacro:macro>
-  <xacro:macro name="robstride_rs02_params" params="can_id kp kd direction:=1 gear_ratio:=1.0 position_offset:=0.0 can_timeout_ticks:=4000 command_position_min:='' command_position_max:='' command_velocity_min:='' command_velocity_max:='' command_effort_min:='' command_effort_max:=''">
+  <xacro:macro name="robstride_rs02_params" params="can_id kp kd direction:=1 gear_ratio:=1.0 position_offset:=0.0 can_timeout_ticks:=0 command_position_min:='' command_position_max:='' command_velocity_min:='' command_velocity_max:='' command_effort_min:='' command_effort_max:=''">
     <param name="model">RS02</param>
     <param name="can_id">${can_id}</param><param name="can_timeout_ticks">${can_timeout_ticks}</param>

Commit message: Support partial operation and recovery gating

File: robstride_examples/description/robstride_example.urdf.xacro (robot description, xacro)
@@ -20,4 +20,5 @@
       <param name="feedback_timeout_ms">3000</param>
       <param name="fail_on_feedback_timeout">false</param>
+      <param name="set_zero_on_activate">false</param>
       <param name="transmit_failure_timeout_ms">1000</param>
       <param name="run_mode_recovery_timeout_ms">0</param>

File: robstride_ros2_control/description/robstride_motor_profiles.xacro (robot description, xacro)
@@ -14,4 +14,11 @@
     <state_interface name="temperature"/>
     <state_interface name="fault"/>
+    <state_interface name="online"/>
+    <state_interface name="ready"/>
+  </xacro:macro>
+  <xacro:macro name="robstride_resilience_params">
+    <param name="feedback_timeout_ms">500</param>
+    <param name="fail_on_feedback_timeout">true</param>
+    <param name="set_zero_on_activate">false</param>
   </xacro:macro>
   <xacro:macro name="robstride_command_limits" params="position_min position_max velocity_min velocity_max effort_min effort_max">
